File: MeowCU/MeowCU.kicad_pcb (KiCad board)
At the start: 4 copper layers, 58.7 x 35.5 mm, 67 parts, among them J1 SWD, J10 Screw_Terminal_01x03, J11 Conn_02x10_Odd_Even, J2 Conn_02x04_Odd_Even, J4 SPI1, J5 5V_IN, J6 OLED, J7 USB_C_Receptacle_USB2.0_16P, J9 PWM, SW6 BTN_UTIL, SW8 BTN_UTIL, SW9 BTN_UTIL, U1 STM32F405RGT6, U2 USBLC6-2SC6, U3 SN65HVD230, U4 AP2112K-3.3, Y1 25MHz

Commit message: V1.7 Release
Parts:
- removed J5: 5V_IN, Connector_PinHeader_2.54mm:PinHeader_1x02_P2.54mm_Vertical
- removed J9: PWM, Connector_PinHeader_2.54mm:PinHeader_2x03_P2.54mm_Vertical
- added J3: Conn_02x03_Odd_Even, Connector_PinSocket_2.54mm:PinSocket_2x03_P2.54mm_Vertical, F.Cu at (159.8, 122.5)
- added R21: 30k, Resistor_SMD:R_0402_1005Metric, F.Cu at (168.1, 116.5)
- added R22: 10k, Resistor_SMD:R_0402_1005Metric, F.Cu at (168.1, 118.1)
- added U5: TPS2116DRL, Package_TO_SOT_SMD:SOT-583-8, F.Cu at (167.8, 114.2)
- J11: footprint Connector_PinHeader_2.54mm:PinHeader_2x10_P2.54mm_Vertical -> Connector_PinSocket_2.54mm:PinSocket_2x10_P2.54mm_Vertical
- J2: value Conn_02x04_Odd_Even -> I2C1/USART3; footprint Connector_PinHeader_2.54mm:PinHeader_2x04_P2.54mm_Vertical -> Connector_PinSocket_2.54mm:PinSocket_2x04_P2.54mm_Vertical
- J4: value SPI1 -> Conn_02x03_Odd_Even; footprint Connector_PinHeader_2.54mm:PinHeader_2x03_P2.54mm_Vertical -> Connector_PinSocket_2.54mm:PinSocket_2x03_P2.54mm_Vertical
- moved J11 2.54 mm to (118.5, 99.0)
- moved J2 2.54 mm to (160.8, 95.0)
- moved J4 2.54 mm to (149.4, 122.5)
- moved R17 1.95 mm to (162.1, 117.4)
- moved C15 1.09 mm to (158.2, 113.9)
- moved C14 1.03 mm to (165.0, 114.1)
- moved D1 0.97 mm to (164.7, 117.4), turned to -90 degrees
- moved U4 0.85 mm to (161.6, 114.2)
- moved R2 0.80 mm to (163.4, 117.4), turned to -90 degrees
- moved C20 0.36 mm to (159.6, 111.4), turned to 180 degrees
Connections:
- C13 pad 1: +5V -> USB_VBUS
- C20 pad 1: +5V -> USB_VBUS
- C24 pad 1: +5V -> USB_VBUS
- J11 pad 10: PC2 -> PC12
- J11 pad 11: PC3 -> PA0
- J11 pad 12: PA0 -> PC3
- J11 pad 13: PA1 -> PC9
- J11 pad 14: PC9 -> PA1
- J11 pad 15: PC8 -> PC7
- J11 pad 16: PC7 -> PC8
- J11 pad 17: PC6 -> PB15
- J11 pad 18: PB15 -> PC6
- J11 pad 19: PB14 -> PB12
- J11 pad 20: PB12 -> PB14
- J11 pad 3: +5V -> EXTERN_5V
- J11 pad 4: +5V -> EXTERN_5V
- J11 pad 7: PB4 -> PB3
- J11 pad 8: PB3 -> PB4
- J11 pad 9: PC12 -> PC2
- J2 pad 5: I2C1_SCL -> USART3_TX
- J2 pad 6: USART3_TX -> I2C1_SCL
- J2 pad 7: I2C1_SDA -> USART3_RX
- J2 pad 8: USART3_RX -> I2C1_SDA
- J4 pad 1: +3.3V -> SPI1_MOSI
- J4 pad 2: SPI1_MOSI -> +3.3V
- J4 pad 3: GND -> SPI1_MISO
- J4 pad 4: SPI1_MISO -> GND
- J4 pad 5: SPI1_CLK -> SPI1_CS
- J4 pad 6: SPI1_CS -> SPI1_CLK
- J6 pad 2: +5V -> EXTERN_5V
- J7 pad A4: +5V -> USB_VBUS
- J7 pad A9: +5V -> USB_VBUS
- J7 pad B4: +5V -> USB_VBUS
- J7 pad B9: +5V -> USB_VBUS
- U2 pad 5: +5V -> USB_VBUS
Routing:
- net +5V: track 102.6 -> 6.47 mm, vias 10 -> 0
- net EXTERN_5V: track 0.00 -> 93.5 mm, vias 0 -> 4
- net USB_VBUS: track 0.00 -> 12.7 mm, vias 0 -> 9
- net +3.3V: track 50.2 -> 46.8 mm
- net Net-(U5-PR1): track 0.00 -> 3.17 mm
- net GND: track 53.0 -> 53.8 mm, vias 56 -> 58
- added copper zone on F.Cu, net EXTERN_5V
- added copper zone on In2.Cu, net EXTERN_5V
- added copper zone on F.Cu, net USB_VBUS
- added copper zone on In2.Cu, net USB_VBUS
- removed copper zone on In2.Cu, net +5V
Other:
- board text added: "2026/10 V1.7"
- board text added: "V1.7"
- board text removed: "2026/10 V1.6"
- board text removed: "5V IN"
- board text removed: "V1.6"
